File: Keyboard.sch (EAGLE design)
At the start: 78 parts

Commit message: Added more to keyboard schematic
Parts:
- added D1, D10, D11, D12, D13, D14, D15, D16, D17, D18, D19, D2, D20, D21, D22, D23, D24, D25, D26, D27, D28, D29, D3, D30, D31, D32, D33, D34, D35, D36, D37, D38, D39, D4, D40, D41, D42, D43, D44, D45, D46, D47, D48, D49, D5, D50, D51, D52, D53, D54, D55, D56, D57, D58, D59, D6, D60, D61, D62, D63, D64, D65, D66, D67, D68, D69, D7, D70, D71, D72, D73, D74, D75, D76, D77, D78, D79, D8, D80, D81, D82, D83, D84, D85, D86, D87, D9: 1N4148DO35-7, diode:1N4148DO35-7
- added F1, F10, F2, F3, F4, F5, F6, F7, F8, F9: CHERRY_MX_LED, cherry:CHERRY_MX_LED
- added U$1: ARDUINO-TEENSY++, teensypp:ARDUINO-TEENSY++
Connections:
- new net N$1: D1.A, NUM_MINUSG$1.2
- new net N$10: D10.A, TOP_5G$1.2
- new net N$100: LEFT_ALTG$1.1, S_KEYG$1.1, TOP_2G$1.1, W_KEYG$1.1, X_KEYG$1.1
- new net N$101: C_KEYG$1.1, D_KEYG$1.1, E_KEYG$1.1, SPACE_BARG$1.1, TOP_3G$1.1
- new net N$102: F_KEYG$1.1, RIGHT_ALTG$1.1, R_KEYG$1.1, TOP_4G$1.1, V_KEYG$1.1
- new net N$103: B_KEYG$1.1, G_KEYG$1.1, RIGHT_WIN_KEYG$1.1, TOP_5G$1.1, T_KEYG$1.1
- new net N$104: H_KEYG$1.1, MENU_KEYG$1.1, N_KEYG$1.1, TOP_6G$1.1, Y_KEYG$1.1
- new net N$105: J_KEYG$1.1, M_KEYG$1.1, RIGHT_CONTROLG$1.1, TOP_7G$1.1, U_KEYG$1.1
- new net N$106: COMMAG$1.1, I_KEYG$1.1, K_KEYG$1.1, TOP_8G$1.1
- new net N$107: L_KEYG$1.1, O_KEYG$1.1, PERIODG$1.1, TOP_9G$1.1
- new net N$108: COLONG$1.1, P_KEYG$1.1, QUESTION_MARKG$1.1, TOP_0G$1.1
- new net N$109: HYPHENG$1.1, LEFT_BRACKETG$1.1, QUOTEG$1.1, RIGHT_SHIFTG$1.1
- new net N$11: D11.A, TOP_6G$1.2
- new net N$110: ENTER_KEYG$1.1, PLUS_EQUALSG$1.1, RIGHT_BRACKETG$1.1
- new net N$111: BACKSLASHG$1.1, BACKSPACEG$1.1
- new net N$112: F1G$1.1, F3G$1.1, F5G$1.1, F7G$1.1, F9G$1.1
- new net N$113: F10G$1.1, F2G$1.1, F4G$1.1, F6G$1.1, F8G$1.1
- new net N$12: D12.A, TOP_7G$1.2
- new net N$13: D13.A, TOP_8G$1.2
- new net N$14: D14.A, TOP_9G$1.2
- new net N$15: D15.A, TOP_0G$1.2
- new net N$16: D16.A, HYPHENG$1.2
- new net N$17: D17.A, PLUS_EQUALSG$1.2
- new net N$18: BACKSPACEG$1.2, D18.A
- new net N$19: D19.A, F1G$1.2
- new net N$2: D2.A, NUM_DIVIDEG$1.2
- new net N$20: D20.A, F2G$1.2
- new net N$21: D21.A, NUM_PLUSG$1.2
- new net N$22: D22.A, NUM_7G$1.2
- new net N$23: D23.A, NUM_8G$1.2
- new net N$24: D24.A, NUM_9G$1.2
- new net N$25: D25.A, TABG$1.2
- new net N$26: D26.A, Q_KEYG$1.2
- new net N$27: D27.A, W_KEYG$1.2
- new net N$28: D28.A, E_KEYG$1.2
- new net N$29: D29.A, R_KEYG$1.2
- new net N$3: D3.A, NUM_MULTIPLYG$1.2
- new net N$30: D30.A, T_KEYG$1.2
- new net N$31: D31.A, Y_KEYG$1.2
- new net N$32: D32.A, U_KEYG$1.2
- new net N$33: D33.A, I_KEYG$1.2
- new net N$34: D34.A, O_KEYG$1.2
- new net N$35: D35.A, P_KEYG$1.2
- new net N$36: D36.A, LEFT_BRACKETG$1.2
- new net N$37: D37.A, RIGHT_BRACKETG$1.2
- new net N$38: BACKSLASHG$1.2, D38.A
- new net N$39: D39.A, F3G$1.2
- new net N$4: D4.A, NUM_LOCKG$1.2
- new net N$40: D40.A, F4G$1.2
- new net N$41: D41.A, NUM_4G$1.2
- new net N$42: D42.A, NUM_5G$1.2
- new net N$43: D43.A, NUM_6G$1.2
- new net N$44: CAPS_LOCKG$1.2, D44.A
- new net N$45: A_KEYG$1.2, D45.A
- new net N$46: D46.A, S_KEYG$1.2
- new net N$47: D47.A, D_KEYG$1.2
- new net N$48: D48.A, F_KEYG$1.2
- new net N$49: D49.A, G_KEYG$1.2
- new net N$5: D5.A, ESCG$1.2
- new net N$50: D50.A, H_KEYG$1.2
- new net N$51: D51.A, J_KEYG$1.2
- new net N$52: D52.A, K_KEYG$1.2
- new net N$53: D53.A, L_KEYG$1.2
- new net N$54: COLONG$1.2, D54.A
- new net N$55: D55.A, QUOTEG$1.2
- new net N$56: D56.A, ENTER_KEYG$1.2
- new net N$57: D57.A, F5G$1.2
- new net N$58: D58.A, F6G$1.2
- new net N$59: D59.A, NUM_ENTERG$1.2
- new net N$6: D6.A, TOP_1G$1.2
- new net N$60: D60.A, NUM_1G$1.2
- new net N$61: D61.A, NUM_2G$1.2
- new net N$62: D62.A, NUM_3G$1.2
- new net N$63: D63.A, LEFT_SHIFTG$1.2
- new net N$64: D64.A, Z_KEYG$1.2
- new net N$65: D65.A, X_KEYG$1.2
- new net N$66: C_KEYG$1.2, D66.A
- new net N$67: D67.A, V_KEYG$1.2
- new net N$68: B_KEYG$1.2, D68.A
- new net N$69: D69.A, N_KEYG$1.2
- new net N$7: D7.A, TOP_2G$1.2
- new net N$70: D70.A, M_KEYG$1.2
- new net N$71: COMMAG$1.2, D71.A
- new net N$72: D72.A, PERIODG$1.2
- new net N$73: D73.A, QUESTION_MARKG$1.2
- new net N$74: D74.A, F7G$1.2
- new net N$75: D75.A, F8G$1.2
- new net N$76: D76.A, NUM_DOTG$1.2
- new net N$77: D77.A, NUM_0G$1.2
- new net N$78: D78.A, LEFT_CONTROLG$1.2
- new net N$79: D79.A, LEFT_WIN_KEYG$1.2
- new net N$8: D8.A, TOP_3G$1.2
- new net N$80: D80.A, LEFT_ALTG$1.2
- new net N$81: D81.A, SPACE_BARG$1.2
- new net N$82: D82.A, RIGHT_ALTG$1.2
- new net N$83: D83.A, RIGHT_WIN_KEYG$1.2
- new net N$84: D84.A, MENU_KEYG$1.2
- new net N$85: D85.A, RIGHT_CONTROLG$1.2
- new net N$86: D86.A, F9G$1.2
- new net N$87: D87.A, F10G$1.2
- new net N$88: D1.C, D10.C, D11.C, D12.C, D13.C, D14.C, D15.C, D16.C, D17.C, D18.C, D19.C, D2.C, D20.C, D3.C, D4.C, D5.C, D6.C, D7.C, D8.C, D9.C
- new net N$9: D9.A, TOP_4G$1.2
- new net N$90: D21.C, D22.C, D23.C, D24.C, D25.C, D26.C, D27.C, D28.C, D29.C, D30.C, D31.C, D32.C, D33.C, D34.C, D35.C, D36.C, D37.C, D38.C, D39.C, D40.C
- new net N$91: D41.C, D42.C, D43.C, D44.C, D45.C, D46.C, D47.C, D48.C, D49.C, D50.C, D51.C, D52.C, D53.C, D54.C, D55.C, D56.C, D57.C, D58.C
- new net N$92: D59.C, D60.C, D61.C, D62.C, D63.C, D64.C, D65.C, D66.C, D67.C, D68.C, D69.C, D70.C, D71.C, D72.C, D73.C, D74.C, D75.C, RIGHT_SHIFTG$1.2
- new net N$93: D76.C, D77.C, D78.C, D79.C, D80.C, D81.C, D82.C, D83.C, D84.C, D85.C, D86.C, D87.C
- new net N$94: NUM_ENTERG$1.1, NUM_MINUSG$1.1, NUM_PLUSG$1.1
- new net N$95: NUM_1G$1.1, NUM_4G$1.1, NUM_7G$1.1, NUM_DIVIDEG$1.1, NUM_DOTG$1.1
- new net N$96: NUM_0G$1.1, NUM_2G$1.1, NUM_5G$1.1, NUM_8G$1.1, NUM_MULTIPLYG$1.1
- new net N$97: NUM_3G$1.1, NUM_6G$1.1, NUM_9G$1.1, NUM_LOCKG$1.1
- new net N$98: CAPS_LOCKG$1.1, ESCG$1.1, LEFT_CONTROLG$1.1, LEFT_SHIFTG$1.1, TABG$1.1
- new net N$99: A_KEYG$1.1, LEFT_WIN_KEYG$1.1, Q_KEYG$1.1, TOP_1G$1.1, Z_KEYG$1.1

Commit message: Added and connected nets
Connections:
- removed net N$100: LEFT_ALTG$1.1, S_KEYG$1.1, TOP_2G$1.1, W_KEYG$1.1, X_KEYG$1.1
- removed net N$101: C_KEYG$1.1, D_KEYG$1.1, E_KEYG$1.1, SPACE_BARG$1.1, TOP_3G$1.1
- removed net N$102: F_KEYG$1.1, RIGHT_ALTG$1.1, R_KEYG$1.1, TOP_4G$1.1, V_KEYG$1.1
- removed net N$103: B_KEYG$1.1, G_KEYG$1.1, RIGHT_WIN_KEYG$1.1, TOP_5G$1.1, T_KEYG$1.1
- removed net N$104: H_KEYG$1.1, MENU_KEYG$1.1, N_KEYG$1.1, TOP_6G$1.1, Y_KEYG$1.1
- removed net N$105: J_KEYG$1.1, M_KEYG$1.1, RIGHT_CONTROLG$1.1, TOP_7G$1.1, U_KEYG$1.1
- removed net N$106: COMMAG$1.1, I_KEYG$1.1, K_KEYG$1.1, TOP_8G$1.1
- removed net N$107: L_KEYG$1.1, O_KEYG$1.1, PERIODG$1.1, TOP_9G$1.1
- removed net N$108: COLONG$1.1, P_KEYG$1.1, QUESTION_MARKG$1.1, TOP_0G$1.1
- removed net N$109: HYPHENG$1.1, LEFT_BRACKETG$1.1, QUOTEG$1.1, RIGHT_SHIFTG$1.1
- removed net N$110: ENTER_KEYG$1.1, PLUS_EQUALSG$1.1, RIGHT_BRACKETG$1.1
- removed net N$111: BACKSLASHG$1.1, BACKSPACEG$1.1
- removed net N$112: F1G$1.1, F3G$1.1, F5G$1.1, F7G$1.1, F9G$1.1
- removed net N$113: F10G$1.1, F2G$1.1, F4G$1.1, F6G$1.1, F8G$1.1
- removed net N$88: D1.C, D10.C, D11.C, D12.C, D13.C, D14.C, D15.C, D16.C, D17.C, D18.C, D19.C, D2.C, D20.C, D3.C, D4.C, D5.C, D6.C, D7.C, D8.C, D9.C
- removed net N$90: D21.C, D22.C, D23.C, D24.C, D25.C, D26.C, D27.C, D28.C, D29.C, D30.C, D31.C, D32.C, D33.C, D34.C, D35.C, D36.C, D37.C, D38.C, D39.C, D40.C
- removed net N$91: D41.C, D42.C, D43.C, D44.C, D45.C, D46.C, D47.C, D48.C, D49.C, D50.C, D51.C, D52.C, D53.C, D54.C, D55.C, D56.C, D57.C, D58.C
- removed net N$92: D59.C, D60.C, D61.C, D62.C, D63.C, D64.C, D65.C, D66.C, D67.C, D68.C, D69.C, D70.C, D71.C, D72.C, D73.C, D74.C, D75.C, RIGHT_SHIFTG$1.2
- removed net N$93: D76.C, D77.C, D78.C, D79.C, D80.C, D81.C, D82.C, D83.C, D84.C, D85.C, D86.C, D87.C
- removed net N$94: NUM_ENTERG$1.1, NUM_MINUSG$1.1, NUM_PLUSG$1.1
- removed net N$95: NUM_1G$1.1, NUM_4G$1.1, NUM_7G$1.1, NUM_DIVIDEG$1.1, NUM_DOTG$1.1
- removed net N$96: NUM_0G$1.1, NUM_2G$1.1, NUM_5G$1.1, NUM_8G$1.1, NUM_MULTIPLYG$1.1
- removed net N$97: NUM_3G$1.1, NUM_6G$1.1, NUM_9G$1.1, NUM_LOCKG$1.1
- removed net N$98: CAPS_LOCKG$1.1, ESCG$1.1, LEFT_CONTROLG$1.1, LEFT_SHIFTG$1.1, TABG$1.1
- removed net N$99: A_KEYG$1.1, LEFT_WIN_KEYG$1.1, Q_KEYG$1.1, TOP_1G$1.1, Z_KEYG$1.1
- new net PINB0: NUM_1G$1.1, NUM_4G$1.1, NUM_7G$1.1, NUM_DIVIDEG$1.1, NUM_DOTG$1.1, U$1.20
- new net PINB1: NUM_ENTERG$1.1, NUM_MINUSG$1.1, NUM_PLUSG$1.1, U$1.21
- new net PINB2: D76.C, D77.C, D78.C, D79.C, D80.C, D81.C, D82.C, D83.C, D84.C, D85.C, D86.C, D87.C, U$1.22
- new net PINB3: D59.C, D60.C, D61.C, D62.C, D63.C, D64.C, D65.C, D66.C, D67.C, D68.C, D69.C, D70.C, D71.C, D72.C, D73.C, D74.C, D75.C, RIGHT_SHIFTG$1.2, U$1.23
- new net PINB4: D41.C, D42.C, D43.C, D44.C, D45.C, D46.C, D47.C, D48.C, D49.C, D50.C, D51.C, D52.C, D53.C, D54.C, D55.C, D56.C, D57.C, D58.C, U$1.24,PWM
- new net PINB5: D21.C, D22.C, D23.C, D24.C, D25.C, D26.C, D27.C, D28.C, D29.C, D30.C, D31.C, D32.C, D33.C, D34.C, D35.C, D36.C, D37.C, D38.C, D39.C, D40.C, U$1.25,PWM
- new net PINB6: D1.C, D10.C, D11.C, D12.C, D13.C, D14.C, D15.C, D16.C, D17.C, D18.C, D19.C, D2.C, D20.C, D3.C, D4.C, D5.C, D6.C, D7.C, D8.C, D9.C, U$1.26,PWM
- new net PINB7: COMMAG$1.1, I_KEYG$1.1, K_KEYG$1.1, TOP_8G$1.1, U$1.27,PWM
- new net PIND0: L_KEYG$1.1, O_KEYG$1.1, PERIODG$1.1, TOP_9G$1.1, U$1.0,PWM,INT0
- new net PIND1: COLONG$1.1, P_KEYG$1.1, QUESTION_MARKG$1.1, TOP_0G$1.1, U$1.1,PWM,INT1
- new net PIND2: HYPHENG$1.1, LEFT_BRACKETG$1.1, QUOTEG$1.1, RIGHT_SHIFTG$1.1, U$1.2,RX,INT2
- new net PIND3: ENTER_KEYG$1.1, PLUS_EQUALSG$1.1, RIGHT_BRACKETG$1.1, U$1.3,TX,INT3
- new net PIND4: BACKSLASHG$1.1, BACKSPACEG$1.1, U$1.4
- new net PIND5: F1G$1.1, F3G$1.1, F5G$1.1, F7G$1.1, F9G$1.1, U$1.5
- new net PIND7: F10G$1.1, F2G$1.1, F4G$1.1, F6G$1.1, F8G$1.1, U$1.7
- new net PINE0: U$1.8
- new net PINE1: U$1.9
- new net PINE6: NUM_3G$1.1, NUM_6G$1.1, NUM_9G$1.1, NUM_LOCKG$1.1, U$1.18,INT6
- new net PINE7: NUM_0G$1.1, NUM_2G$1.1, NUM_5G$1.1, NUM_8G$1.1, NUM_MULTIPLYG$1.1, U$1.19
- new net PINF0: CAPS_LOCKG$1.1, ESCG$1.1, LEFT_CONTROLG$1.1, LEFT_SHIFTG$1.1, TABG$1.1, U$1.38,A0
- new net PINF1: A_KEYG$1.1, LEFT_WIN_KEYG$1.1, Q_KEYG$1.1, TOP_1G$1.1, U$1.39,A1, Z_KEYG$1.1
- new net PINF2: LEFT_ALTG$1.1, S_KEYG$1.1, TOP_2G$1.1, U$1.40,A2, W_KEYG$1.1, X_KEYG$1.1
- new net PINF3: C_KEYG$1.1, D_KEYG$1.1, E_KEYG$1.1, SPACE_BARG$1.1, TOP_3G$1.1, U$1.41,A3
- new net PINF4: F_KEYG$1.1, RIGHT_ALTG$1.1, R_KEYG$1.1, TOP_4G$1.1, U$1.42,A4, V_KEYG$1.1
- new net PINF5: B_KEYG$1.1, G_KEYG$1.1, RIGHT_WIN_KEYG$1.1, TOP_5G$1.1, T_KEYG$1.1, U$1.43,A5
- new net PINF6: H_KEYG$1.1, MENU_KEYG$1.1, N_KEYG$1.1, TOP_6G$1.1, U$1.44,A6, Y_KEYG$1.1
- new net PINF7: J_KEYG$1.1, M_KEYG$1.1, RIGHT_CONTROLG$1.1, TOP_7G$1.1, U$1.45,A7, U_KEYG$1.1
