File: AutoGenerateCadFiles/GeneratedKeyboard.brd (EAGLE design)
At the start: 387 x 104 mm, 167 parts

Commit message: Fixed an issue where 2 columns were connected together
Parts:
- moved _1 96.2 mm to (183.5, 11.3)
- moved 0 96.1 mm to (281.2, 86.5)
- moved 1 96.1 mm to (109.8, 86.5)
- moved 2 96.1 mm to (128.8, 86.5)
- moved 3 96.1 mm to (147.9, 86.5)
- moved 4 96.1 mm to (166.9, 86.5)
- moved 5 96.1 mm to (186.0, 86.5)
- moved 6 96.1 mm to (205.0, 86.5)
- moved 7 96.1 mm to (224.1, 86.5)
- moved 8 96.1 mm to (243.1, 86.5)
- moved 9 96.1 mm to (262.2, 86.5)
- moved A 96.1 mm to (124.1, 48.4)
- moved ALT 96.1 mm to (140.7, 10.3)
- moved ALT2 96.1 mm to (283.6, 10.3)
- moved B 96.1 mm to (209.8, 29.3)
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Connections:
- net PINC6: now also KP_1.MX1, KP_4.MX1, KP_7.MX1, KP_DEL.MX1, KP_SLASH.MX1; no longer ENTER2.MX1, EQUAL2.MX1, KP_DASH.MX1
- net PINC7: now also ENTER2.MX1, EQUAL2.MX1, KP_DASH.MX1
- net PIND3: no longer CAPSLOCK.MX1, CTRL.MX1, ESC.MX1, SHIFT.MX1, TAB.MX1
- net PIND4: now also CAPSLOCK.MX1, CTRL.MX1, ESC.MX1, SHIFT.MX1, TAB.MX1; no longer KP_0.MX1, KP_3.MX1, KP_6.MX1, KP_9.MX1, NUMLOCK.MX1
- net PIND5: now also KP_0.MX1, KP_3.MX1, KP_6.MX1, KP_9.MX1, NUMLOCK.MX1; no longer KP_2.MX1, KP_5.MX1, KP_8.MX1, KP_ASTERISK.MX1
- net PIND7: now also KP_2.MX1, KP_5.MX1, KP_8.MX1, KP_ASTERISK.MX1; no longer KP_1.MX1, KP_4.MX1, KP_7.MX1, KP_DEL.MX1, KP_SLASH.MX1
Routing:
- net PINC7: track 0.00 -> 266.8 mm, vias 0 -> 2
- net PIND3: track 227.8 -> 158.3 mm, vias 0 -> 1
- net PIND7: track 249.3 -> 213.5 mm
- net PINB3: track 440.4 -> 416.4 mm, vias 0 -> 1
- net PIND4: track 210.6 -> 193.2 mm
- net PINC6: track 250.6 -> 239.1 mm
- net PINE6: track 291.7 -> 281.1 mm, vias 1 -> 2
- net PINB4: track 407.5 -> 397.9 mm
- net PIND1: track 121.4 -> 112.0 mm
- net PIND5: track 233.0 -> 223.8 mm
- net PINB7: track 281.0 -> 272.3 mm
- net PIND0: track 109.3 -> 117.5 mm
- net PINB1: track 493.4 -> 485.8 mm, vias 0 -> 1
- net PIND2: track 140.7 -> 148.0 mm
- net PINB6: track 281.1 -> 273.9 mm
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Other:
- board size 387 x 104 mm -> 387 x 101 mm
