File: CAD Files Try 2/KeyboardWithArrows.brd (EAGLE design)
At the start: 386 x 98 mm, 169 parts

Commit message: Fixed part of board where a key was missing a connection
Parts:
- flipped J to the top
Connections:
- new net N$84: DEQUAL2.A, EQUAL2.MX2
Routing:
- net PINB0: track 259.3 -> 288.9 mm, vias 0 -> 1
- net PINB3: track 192.6 -> 166.5 mm
- net PINB1: track 225.6 -> 249.0 mm, vias 0 -> 1
- net PIND2: track 403.3 -> 412.1 mm, vias 0 -> 2
- net PIND0: track 465.6 -> 473.3 mm
- net PINC7: track 251.3 -> 244.3 mm
- net PINB7: track 88.0 -> 94.7 mm
- net N$84: track 0.00 -> 6.49 mm
- net PINB5: track 133.5 -> 139.7 mm, vias 0 -> 1
- net PINF7: track 189.2 -> 194.6 mm
- net PINB4: track 143.5 -> 138.4 mm, vias 1 -> 2
- net N$48: track 11.6 -> 6.58 mm
- net PIND1: track 446.5 -> 450.6 mm
- net PIND3: track 408.5 -> 405.1 mm, vias 0 -> 1
- net PINF0: track 112.8 -> 115.8 mm
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